File: KiCAD/PC8001-YM2203.sch (KiCad schematic (older format))
At the start: 29 parts, among them J1 PC-8001 ext BUS, J2 ADDR JP, J3 OUTPUT, U1 NJM5532DD, U2 74HC32, U3 74HC138, U4 DLO555MB, U5 YM2203, U6 YM3014B

Commit message: 74HC32、HC138は74LS32、LS138の間違いだったので修正
Parts:
- U2: value 74HC32 -> 74LS32
- U3: value 74HC138 -> 74LS138
Changed lines of the file:
@@
 P 3650 3900
 F 0 "U2" H 3650 3900 50  0000 C CNN
-F 1 "74HC32" H 3650 4134 50  0000 C CNN
+F 1 "74LS32" H 3650 4134 50  0000 C CNN
 F 2 "" H 3650 3900 50  0001 C CNN
 F 3 "http://www.ti.com/lit/gpn/sn74LS32" H 3650 3900 50  0001 C CNN
@@
 P 3650 3450
 F 0 "U2" H 3650 3450 50  0000 C CNN
-F 1 "74HC32" H 3650 3684 50  0000 C CNN
+F 1 "74LS32" H 3650 3684 50  0000 C CNN
 F 2 "" H 3650 3450 50  0001 C CNN
 F 3 "http://www.ti.com/lit/gpn/sn74LS32" H 3650 3450 50  0001 C CNN
@@
 P 3350 2100
 F 0 "U3" H 3100 2550 50  0000 C CNN
-F 1 "74HC138" H 3500 2550 50  0000 C CNN
+F 1 "74LS138" H 3500 2550 50  0000 C CNN
 F 2 "" H 3350 2100 50  0001 C CNN
 F 3 "http://www.ti.com/lit/gpn/sn74LS138" H 3350 2100 50  0001 C CNN
@@
 P 2050 4500
 F 0 "U2" H 2050 4500 50  0000 C CNN
-F 1 "74HC32" H 2050 4734 50  0000 C CNN
+F 1 "74LS32" H 2050 4734 50  0000 C CNN
 F 2 "" H 2050 4500 50  0001 C CNN
 F 3 "http://www.ti.com/lit/gpn/sn74LS32" H 2050 4500 50  0001 C CNN
@@
 P 2050 5000
 F 0 "U2" H 2050 5000 50  0000 C CNN
-F 1 "74HC32" H 2050 5234 50  0000 C CNN
+F 1 "74LS32" H 2050 5234 50  0000 C CNN
 F 2 "" H 2050 5000 50  0001 C CNN
 F 3 "http://www.ti.com/lit/gpn/sn74LS32" H 2050 5000 50  0001 C CNN
@@
 P 2150 6750
 F 0 "U2" H 2150 6750 50  0000 C CNN
-F 1 "74HC32" H 2400 6400 50  0000 C CNN
+F 1 "74LS32" H 2400 6400 50  0000 C CNN
 F 2 "" H 2150 6750 50  0001 C CNN
 F 3 "http://www.ti.com/lit/gpn/sn74LS32" H 2150 6750 50  0001 C CNN

Commit message: I/O端子設置、プリントパターン検討
Parts:
- removed J3: OUTPUT, symbol Connector:AudioJack2_Ground_Switch
- added J3: Audio-Jack-3_2Switches, AJ-1780:AJ-1780, symbol PC8001-YM2203-rescue:Audio-Jack-3_2Switches-YM2151-rescue
- added J4: A-CON, Connector_PinHeader_2.54mm:PinHeader_2x07_P2.54mm_Vertical, symbol Connector_Generic:Conn_02x07_Odd_Even
- added J5: B-CON, Connector_PinHeader_2.54mm:PinHeader_2x07_P2.54mm_Vertical, symbol Connector_Generic:Conn_02x07_Odd_Even
- added NT1: Net-Tie_2, NetTie:NetTie-2_SMD_Pad2.0mm, symbol Device:Net-Tie_2
- C1, C7, C8, C9: footprint (none) -> Capacitor_THT:CP_Radial_D5.0mm_P2.50mm
- C2, C3, C4, C5, C6: footprint (none) -> Capacitor_THT:C_Disc_D3.0mm_W1.6mm_P2.50mm
- H1, H2, H3, H4: footprint (none) -> MountingHole:MountingHole_3.2mm_M3
- J1: footprint (none) -> Connector_PinHeader_2.54mm:PinHeader_2x25_P2.54mm_Horizontal
- J2: footprint (none) -> Connector_PinHeader_2.54mm:PinHeader_2x08_P2.54mm_Vertical
- R1, R2, R3, R4, R5: footprint (none) -> Resistor_THT:R_Axial_DIN0207_L6.3mm_D2.5mm_P10.16mm_Horizontal
- RV1, RV2: footprint (none) -> Potentiometer_THT:Potentiometer_Vishay_T73YP_Vertical
- U1, U6: footprint (none) -> Package_DIP:DIP-8_W7.62mm_Socket
- U2: footprint (none) -> Package_DIP:DIP-14_W7.62mm_Socket
- U3: footprint (none) -> Package_DIP:DIP-16_W7.62mm_Socket
- U4: footprint (none) -> Package_TO_SOT_THT:TO-92_Inline_Wide
- U5: footprint (none) -> Package_DIP:DIP-40_W15.24mm_Socket
Connections:
- net GND: now also J4.14 (Pin_14), J5.14 (Pin_14), NT1.2; no longer C2.1, C6.1, C8.2, RV1.3, RV2.3, U1.4 (V-), U5.17 (AGND), U6.6 (GND)
- net VCC: now also J4.13 (Pin_13), J5.13 (Pin_13)
- net IOA6: now reaches U5.10 (IOA6)
- net IOA6: now also J4.7 (Pin_7)
- net IOA5: now reaches U5.11 (IOA5)
- net IOA5: now also J4.6 (Pin_6)
- net IOA4: now reaches U5.12 (IOA4)
- net IOA4: now also J4.5 (Pin_5)
- net IOA3: now reaches U5.13 (IOA3)
- net IOA3: now also J4.4 (Pin_4)
- net IOA2: now reaches U5.14 (IOA2)
- net IOA2: now also J4.3 (Pin_3)
- net IOA1: now reaches U5.15 (IOA1)
- net IOA1: now also J4.2 (Pin_2)
- net IOA0: now reaches U5.16 (IOA0)
- net IOA0: now also J4.1 (Pin_1)
- net ~IRQ: now reaches U5.25 (~IRQ)
- net ~IRQ: now also J4.12 (Pin_12), J5.12 (Pin_12)
- net IOB0: now reaches U5.26 (IOB0)
- net IOB0: now also J5.1 (Pin_1)
- net IOB1: now reaches U5.27 (IOB1)
- net IOB1: now also J5.2 (Pin_2)
- net IOB2: now reaches U5.28 (IOB2)
- net IOB2: now also J5.3 (Pin_3)
- net IOB3: now reaches U5.29 (IOB3)
- net IOB3: now also J5.4 (Pin_4)
- net IOB4: now reaches U5.30 (IOB4)
- net IOB4: now also J5.5 (Pin_5)
- net IOB5: now reaches U5.31 (IOB5)
- net IOB5: now also J5.6 (Pin_6)
- net IOB6: now reaches U5.32 (IOB6)
- net IOB6: now also J5.7 (Pin_7)
- net IOB7: now reaches U5.33 (IOB7)
- net IOB7: now also J5.8 (Pin_8)
- net IOA7: now reaches U5.9 (IOA7)
- net IOA7: now also J4.8 (Pin_8)
- net at R4.1, R5.1: now also J3.2, J3.5
- new net GNDA: C2.1, C6.1, C8.2, J3.1, NT1.1, RV1.3, RV2.3, U1.4 (V-), U5.17 (AGND), U6.6 (GND)
- no-connect marks 51 -> 40
